Commit message: Add map

File: urdf/udacity_bot.xacro (robot description, xacro)
@@ -1,4 +1,5 @@
 <?xml version='1.0'?>
 <robot name="udacity_bot" xmlns:xacro="http://www.ros.org/wiki/xacro">
+	<xacro:include filename="$(find udacity_bot)/urdf/udacity_bot.gazebo" />
 	<link name="robot_footprint"></link>
 	<joint name="robot_footprint_joint" type="fixed">
@@ -117,3 +118,61 @@
 		</visual>
   	</link>
+  	<joint type="fixed" name="camera_joint">
+  		<origin xyz="0.2 0 0" rpy="0 0 0"/>
+  		<parent link="chassis" />
+  		<child link="camera" />
+  		<axis xyz="0 1 0" rpy="0 0 0"/>
+  	</joint>
+  	<link name="camera">
+  		<inertial>
+  			<mass value="0.1" />
+			<origin xyz="0 0 0" rpy="0 0 0" />
+  			<inertia
+				ixx="1e-6" ixy="0" ixz="0"
+				iyy="1e-6" iyz="0"
+				izz="1e-7"
+			/>
+  		</inertial>
+  		<collision name='camera_collision'>
+			<origin xyz="0 0 0" rpy="0 0 0" />
+			<geometry>
+				<box size=".05 .05 .05" />
+			</geometry>
+		</collision>
+		<visual name="camera_visual">
+			<origin xyz="0 0 0" rpy="0 0 0" />
+			<geometry>
+				<box size=".05 .05 .05" />
+			</geometry>
+		</visual>
+  	</link>
+  	<joint type="fixed" name="hokuyo_joint">
+  		<origin xyz="0.15 0 0.1" rpy="0 0 0"/>
+  		<parent link="chassis" />
+  		<child link="hokuyo" />
+  		<axis xyz="0 1 0" rpy="0 0 0"/>
+  	</joint>
+  	<link name="hokuyo">
+  		<inertial>
+  			<mass value="0.1" />
+			<origin xyz="0 0 0" rpy="0 0 0" />
+  			<inertia
+				ixx="1e-6" ixy="0" ixz="0"
+				iyy="1e-6" iyz="0"
+				izz="1e-7"
+			/>
+  		</inertial>
+  		<collision name='hokuyo_collision'>
+			<origin xyz="0 0 0" rpy="0 0 0" />
+			<geometry>
+				<box size=".1 .1 .1" />
+			</geometry>
+		</collision>
+		<visual name="hokuyo_visual">
+			<origin xyz="0 0 0" rpy="0 0 0" />
+			<geometry>
+				<mesh filename="package://udacity_bot/meshes/hokuyo.dae"/>
+			</geometry>
+		</visual>
+  	</link>
 </robot>
